Commit message: add launch simulation

File: description/robot_core.xacro (robot description, xacro)
@@ -25,5 +25,5 @@
     <link name="chassis">
         <visual>
-        <origin xyz="0.115 0.0 0.0375"/>
+        <origin xyz="0.15 0.0 0.0375"/>
             <geometry>
                 <box size="0.23 0.15 0.075"/>
@@ -32,5 +32,5 @@
         </visual>
         <collision>
-        <origin xyz="0.115 0.0 0.0375"/>
+            <origin xyz="0.15 0.0 0.0375"/>
             <geometry>
                 <box size="0.23 0.15 0.075"/>
@@ -39,7 +39,10 @@
         </collision>
         <xacro:inertial_box mass="0.5" x="0.3" y="0.3" z="0.15">
-            <origin xyz="0.115 0 0.0375" rpy="0 0 0"/>
+            <origin xyz="0.15 0 0.0375" rpy="0 0 0"/>
         </xacro:inertial_box>
     </link>
+    <gazebo reference="chassis">
+        <material>Gazebo/White</material>
+    </gazebo>
     <!-- left wheel link -->
     <joint name="left_wheel_joint" type="continuous">
@@ -65,4 +68,7 @@
         </xacro:inertial_cylinder>
     </link>
+    <gazebo reference="left_wheel">
+        <material>Gazebo/Blue</material>
+    </gazebo>
     <!-- right wheel link -->
     <joint name="right_wheel_joint" type="continuous">
@@ -88,9 +94,12 @@
         </xacro:inertial_cylinder>
     </link>
+    <gazebo reference="right_wheel">
+        <material>Gazebo/Blue</material>
+    </gazebo>
     <!-- caster wheel link -->
     <joint name="caster_wheel_joint" type="fixed">
         <parent link="chassis"/>
         <child link="caster_wheel"/>
-        <origin xyz="0.18 0.0 0.0"/>
+        <origin xyz="0.22 0.0 -0.006"/>
     </joint>
     <link name="caster_wheel">
@@ -110,3 +119,8 @@
         </xacro:inertial_sphere>
     </link>
+    <gazebo reference="caster_wheel">
+        <material>Gazebo/White</material>
+        <mu1 value="0.001"/>
+        <mu2 value="0.001"/>
+    </gazebo>
 </robot>
