Commit message: add sim, 3d

File: description/camera.xacro (robot description, xacro)
@@ -4,5 +4,5 @@
         <parent link="chassis"/>
         <child link="camera_link"/>
-        <origin xyz="0.262 0 0.055" rpy = "0 0 0"/>
+        <origin xyz="0.17 0 0.085" rpy = "0 0 0"/>
     </joint>
     <link name="camera_link">

File: description/lidar.xacro (robot description, xacro)
@@ -4,12 +4,13 @@
         <parent link="chassis"/>
         <child link="laser_frame"/>
-        <origin xyz="0.22 0 0.085" rpy = "0 0 0"/>
+        <origin xyz="0.065 0 0.125" rpy = "0 0 0"/>
     </joint>
     <link name="laser_frame">
         <visual>
             <geometry>
-                <cylinder radius="0.031" length="0.025"/>
+                <!-- <cylinder radius="0.031" length="0.025"/> -->
+                <mesh filename="file://$(find diff_robot)/meshes/sensors/rplidar-a1.stl" scale="0.001 0.001 0.001"/>
             </geometry>
-            <material name="red"/>
+            <material name="black"/>
         </visual>
         <collision>
@@ -23,5 +24,5 @@
     </link>
     <gazebo reference="laser_frame">
-        <material>Gazebo/Red</material>
+        <material>Gazebo/Black</material>
         <sensor name="laser" type="ray">
             <pose> 0 0 0 0 0 0 </pose>

File: description/robot.urdf.xacro (robot description, xacro)
@@ -1,13 +1,13 @@
 <?xml version="1.0"?>
 <robot xmlns:xacro="http://www.ros.org/wiki/xacro"  name="robot">
-     <xacro:arg name="use_ros2_control" default="true"/>
     <xacro:include filename="robot_core.xacro" />
-    <xacro:if value="$(arg use_ros2_control)">
+    <!-- <xacro:if value="$(arg use_ros2_control)">
         <xacro:include filename="ros2_control.xacro" />
     </xacro:if>
     <xacro:unless value="$(arg use_ros2_control)">
         <xacro:include filename="gazebo_control.xacro" />
-    </xacro:unless>
-    <xacro:include filename="lidar.xacro"/>
+    </xacro:unless> -->
+    <xacro:include filename="gazebo_control.xacro" />
+    <!-- <xacro:include filename="lidar.xacro"/> -->
     <xacro:include filename="camera.xacro"/>
 </robot>

File: description/robot_core.xacro (robot description, xacro)
@@ -1,20 +1,25 @@
 <?xml version="1.0"?>
 <robot xmlns:xacro="http://www.ros.org/wiki/xacro">
-    <xacro:include filename="inertial_macros.xacro"/>
-    <material name="white">
-        <color rgba="1 1 1 1"/>
-    </material>
-     <material name="orange">
-        <color rgba="1 0.3 0.1 1"/>
-    </material>
-    <material name="blue">
-        <color rgba="0.2 0.2 1 1"/>
-    </material>
-    <material name="black">
-        <color rgba="0 0 0 1"/>
-    </material>
-    <material name="red">
-        <color rgba="1 0 0 1"/>
-    </material>
+    <xacro:property name="package_name" value="diff_robot" />
+    <xacro:property name="robot_name" value="andino" />
+    <xacro:include filename="$(find ${package_name})/description/common_macros.urdf.xacro" />
+    <xacro:include filename="$(find ${package_name})/description/common_sensors.urdf.xacro" />
+    <xacro:include filename="$(find ${package_name})/description/andino_caster_macro.urdf.xacro" />
+    <xacro:arg name="use_ros2_control" default="true" />
+    <xacro:arg name="sim_mode" default="false" />
+    <xacro:arg name="yaml_config_dir" default="$(find ${package_name})/config/${robot_name}" />
+    <xacro:property name="caster_wheel_yaml" value="$(arg yaml_config_dir)/caster_wheel.yaml" />
+    <xacro:property name="caster_wheel_props" value="${xacro.load_yaml(caster_wheel_yaml)}" />
+    <xacro:arg name="use_fixed_caster" default="True" />
+    <xacro:arg name="use_real_ros_control" default="True" />
+    <xacro:property name="base_yaml" value="$(arg yaml_config_dir)/base.yaml" />
+    <xacro:property name="base_props" value="${xacro.load_yaml(base_yaml)}"/>
+    <xacro:property name="wheel_yaml" value="$(arg yaml_config_dir)/wheel.yaml" />
+    <xacro:property name="wheel_props" value="${xacro.load_yaml(wheel_yaml)}" />
+    <xacro:property name="sensor_yaml" value="$(arg yaml_config_dir)/sensors.yaml" />
+    <xacro:property name="sensor_prop" value="${xacro.load_yaml(sensor_yaml)}" />
+    <xacro:include filename="inertial_macros.xacro" />
+    <!-- Footprint -->
+    <xacro:footprint wheel_props="${wheel_props}" />
     <!-- Base link -->
     <link name="base_link">
@@ -22,25 +27,25 @@
     <!-- Chassis link -->
     <joint name="chassis" type="fixed">
-        <parent link="base_link"/>
-        <child link="chassis"/>
-        <origin xyz="-0.1 0.0 0.0"/>
+        <parent link="base_link" />
+        <child link="chassis" />
+        <origin xyz="-0.1 0.0 0.0" />
     </joint>
     <link name="chassis">
         <visual>
-        <origin xyz="0.15 0.0 0.0375"/>
+            <origin xyz="0.05 0.0 0.075" />
             <geometry>
-                <box size="0.23 0.15 0.075"/>
+                <box size="0.23 0.15 0.075" />
             </geometry>
-            <material name="white"/>
+            <material name="white" />
         </visual>
         <collision>
-            <origin xyz="0.15 0.0 0.0375"/>
+            <origin xyz="0.05 0.0 0.075" />
             <geometry>
-                <box size="0.23 0.15 0.075"/>
+                <box size="0.23 0.15 0.075" />
             </geometry>
-            <material name="white"/>
+            <material name="white" />
         </collision>
         <xacro:inertial_box mass="0.5" x="0.3" y="0.3" z="0.15">
-            <origin xyz="0.15 0 0.0375" rpy="0 0 0"/>
+            <origin xyz="0.05 0 0.075" rpy="0 0 0" />
         </xacro:inertial_box>
     </link>
@@ -48,82 +53,96 @@
         <material>Gazebo/White</material>
     </gazebo>
+    <!-- Wheels -->
+    <xacro:wheel prefix="right" reflect="-1"
+        wheel_props="${wheel_props}"
+        base_props="${base_props}">
+    </xacro:wheel>
+    <xacro:wheel prefix="left" reflect="1"
+        wheel_props="${wheel_props}"
+        base_props="${base_props}">
+    </xacro:wheel>
     <!-- left wheel link -->
-    <joint name="left_wheel_joint" type="continuous">
-        <parent link="base_link"/>
-        <child link="left_wheel"/>
-        <origin xyz="0 0.1 0.0" rpy="-${pi/2} 0 0"/>
-        <axis xyz="0 0 1"/>
+    <!-- <joint name="left_wheel_joint" type="continuous">
+        <parent link="base_link" />
+        <child link="left_wheel" />
+        <origin xyz="0 0.1 0.0" rpy="-${pi/2} 0 0" />
+        <axis xyz="0 0 1" />
     </joint>
     <link name="left_wheel">
         <visual>
             <geometry>
-                <cylinder radius="0.031" length="0.025"/>
+                <cylinder radius="0.031" length="0.025" />
             </geometry>
-            <material name="blue"/>
+            <material name="blue" />
         </visual>
         <collision>
             <geometry>
-                <sphere radius="0.031"/>
+                <sphere radius="0.031" />
             </geometry>
         </collision>
         <xacro:inertial_cylinder mass="0.1" length="0.025" radius="0.031">
-            <origin xyz="0 0 0" rpy="0 0 0"/>
+            <origin xyz="0 0 0" rpy="0 0 0" />
         </xacro:inertial_cylinder>
     </link>
     <gazebo reference="left_wheel">
         <material>Gazebo/Blue</material>
-    </gazebo>
+    </gazebo> -->
     <!-- right wheel link -->
-    <joint name="right_wheel_joint" type="continuous">
-        <parent link="base_link"/>
-        <child link="right_wheel"/>
-        <origin xyz="0 -0.1 0.0" rpy="${pi/2} 0 0"/>
-        <axis xyz="0 0 -1"/>
+    <!-- <joint name="right_wheel_joint" type="continuous">
+        <parent link="base_link" />
+        <child link="right_wheel" />
+        <origin xyz="0 -0.1 0.0" rpy="${pi/2} 0 0" />
+        <axis xyz="0 0 -1" />
     </joint>
     <link name="right_wheel">
         <visual>
             <geometry>
-                <cylinder radius="0.031" length="0.025"/>
+                <cylinder radius="0.031" length="0.025" />
             </geometry>
-            <material name="blue"/>
+            <material name="blue" />
         </visual>
         <collision>
             <geometry>
-                <sphere radius="0.031"/>
+                <sphere radius="0.031" />
             </geometry>
         </collision>
         <xacro:inertial_cylinder mass="0.1" length="0.025" radius="0.031">
-            <origin xyz="0 0 0" rpy="0 0 0"/>
+            <origin xyz="0 0 0" rpy="0 0 0" />
         </xacro:inertial_cylinder>
     </link>
     <gazebo reference="right_wheel">
         <material>Gazebo/Blue</material>
-    </gazebo>
+    </gazebo> -->
     <!-- caster wheel link -->
-    <joint name="caster_wheel_joint" type="fixed">
-        <parent link="chassis"/>
-        <child link="caster_wheel"/>
-        <origin xyz="0.22 0.0 -0.006"/>
+    <!-- <joint name="caster_wheel_joint" type="fixed">
+        <parent link="chassis" />
+        <child link="caster_wheel" />
+        <origin xyz="-0.03 0.0 -0.003" />
     </joint>
     <link name="caster_wheel">
         <visual>
             <geometry>
-                <sphere radius="0.025"/>
+                <sphere radius="0.035" />
             </geometry>
-            <material name="black"/>
+            <material name="black" />
         </visual>
         <collision>
             <geometry>
-                <sphere radius="0.025"/>
+                <sphere radius="0.025" />
             </geometry>
         </collision>
         <xacro:inertial_sphere mass="0.1" radius="0.025">
-            <origin xyz="0 0 0" rpy="0 0 0"/>
+            <origin xyz="0 0 0" rpy="0 0 0" />
         </xacro:inertial_sphere>
     </link>
     <gazebo reference="caster_wheel">
         <material>Gazebo/White</material>
-        <mu1 value="0.001"/>
-        <mu2 value="0.001"/>
-    </gazebo>
+        <mu1 value="0.001" />
+        <mu2 value="0.001" />
+    </gazebo> -->
+    <xacro:caster_wheel reflect="-1" use_fixed="$(arg use_fixed_caster)"
+        wheel_props="${caster_wheel_props}">
+    </xacro:caster_wheel>
+    <xacro:laser prefix="rplidar" parent_link="chassis" sensor_prop="${sensor_prop}">
+    </xacro:laser>
 </robot>

File: description/ros2_control.xacro (robot description, xacro)
@@ -1,29 +1,68 @@
 <?xml version="1.0"?>
 <robot xmlns:xacro="http://www.ros.org/wiki/xacro">
-    <ros2_control name="GazeboSystem" type="system">
-        <hardware>
-            <plugin>gazebo_ros2_control/GazeboSystem</plugin>
-        </hardware>
-        <joint name="left_wheel_joint">
-            <command_interface name="velocity">
-                <param name="min">-10</param>
-                <param name="max">10</param>
-            </command_interface>
-            <state_interface name="velocity"/>
-            <state_interface name="position"/>
-        </joint>
-        <joint name="right_wheel_joint">
-            <command_interface name="velocity">
-                <param name="min">-10</param>
-                <param name="max">10</param>
-            </command_interface>
-            <state_interface name="velocity"/>
-            <state_interface name="position"/>
-        </joint>
-    </ros2_control>
+     <xacro:unless value="$(arg sim_mode)">
+        <ros2_control name="RealRobot" type="system">
+            <hardware>
+                <plugin>diffdrive_arduino/DiffDriveArduino</plugin>
+                <param name="left_wheel_name">left_wheel_joint</param>
+                <param name="right_wheel_name">right_wheel_joint</param>
+                <param name="loop_rate">30</param>
+                <param name="device">/dev/ttyUSB0</param>
+                <param name="baud_rate">57600</param>
+                <param name="timeout">1000</param>
+                <param name="enc_counts_per_rev">525</param>
+            </hardware>
+            <joint name="left_wheel_joint">
+                <command_interface name="velocity">
+                    <param name="min">-5</param>
+                    <param name="max">5</param>
+                </command_interface>
+                <state_interface name="velocity"/>
+                <state_interface name="position"/>
+            </joint>
+            <joint name="right_wheel_joint">
+                <command_interface name="velocity">
+                    <param name="min">-5</param>
+                    <param name="max">5</param>
+                </command_interface>
+                <state_interface name="velocity"/>
+                <state_interface name="position"/>
+            </joint>
+        </ros2_control>
+    </xacro:unless>
+    <xacro:if value="$(arg sim_mode)">
+        <ros2_control name="GazeboSystem" type="system">
+            <hardware>
+                <plugin>gazebo_ros2_control/GazeboSystem</plugin>
+            </hardware>
+            <joint name="left_wheel_joint">
+                <command_interface name="velocity">
+                    <param name="min">-5</param>
+                    <param name="max">5</param>
+                </command_interface>
+                <state_interface name="velocity"/>
+                <state_interface name="position"/>
+            </joint>
+            <joint name="right_wheel_joint">
+                <command_interface name="velocity">
+                    <param name="min">-5</param>
+                    <param name="max">5</param>
+                </command_interface>
+                <state_interface name="velocity"/>
+                <state_interface name="position"/>
+            </joint>
+        </ros2_control>
+    </xacro:if>
+    <gazebo>
+        <plugin name="gazebo_ros2_control" filename="libgazebo_ros2_control.so">
+            <parameters>$(find diff_robot)/config/my_controllers.yaml</parameters>
+            <parameters>$(find diff_robot)/config/gaz_ros2_ctl_use_sim.yaml</parameters>
+        </plugin>
+    </gazebo>
+<!--
     <gazebo>
         <plugin name="gazebo_ros2_control" filename="libgazebo_ros2_control.so">
             <parameters>$(find diff_robot)/config/my_controllers.yaml</parameters>
         </plugin>
-    </gazebo>
+    </gazebo> -->
 </robot>
