Commit message: edit launch_robot

File: description/andino_caster_macro.urdf.xacro (robot description, xacro)
@@ -62,5 +62,5 @@
         xyz="${wheel_props['base']['dx']} ${-wheel_props['base']['dy'] * locationright} ${wheel_props['base']['dz']}"
         rpy="0 0 0" />
-      <parent link="base_link" />
+      <parent link="chassis" />
       <child link="caster_base_link" />
       <axis xyz="0 0 1" />
@@ -115,5 +115,5 @@
           xyz="${wheel_props['hub']['dx']} ${-wheel_props['hub']['dy'] * locationright} ${wheel_props['hub']['dz']}"
           rpy="0 0 0" />
-        <parent link="base_link" />
+        <parent link="chassis" />
         <child link="caster_rotation_link" />
         <axis xyz="0 0 1" />
@@ -126,5 +126,5 @@
           xyz="${wheel_props['hub']['dx']} ${-wheel_props['hub']['dy'] * locationright} ${wheel_props['hub']['dz']}"
           rpy="0 0 0" />
-        <parent link="base_link" />
+        <parent link="chassis" />
         <child link="caster_rotation_link" />
         <axis xyz="0 0 1" />

File: description/common_macros.urdf.xacro (robot description, xacro)
@@ -225,20 +225,20 @@
   - r [float]: sphere radius;
 -->
-  <xacro:macro name="sphere_inertia" params="m r">
+  <!-- <xacro:macro name="sphere_inertia" params="m r">
     <inertial>
       <mass value="${m}"/>
       <inertia ixx="${2.0*m*(r*r)/5.0}" ixy="0.0" ixz="0.0" iyy="${2.0*m*(r*r)/5.0}" iyz="0.0" izz="${2.0*m*(r*r)/5.0}"/>
     </inertial>
-  </xacro:macro>
+  </xacro:macro> -->
 <!-- ===================== Default intertial xacro =============================
   params:
   - m [float]: link mass;
 -->
-  <xacro:macro name="default_inertial" params="mass">
+  <!-- <xacro:macro name="default_inertial" params="mass">
     <inertial>
       <mass value="${mass}"/>
       <inertia ixx="1.0" ixy="0.0" ixz="0.0" iyy="1.0" iyz="0.0" izz="1.0"/>
     </inertial>
-  </xacro:macro>
+  </xacro:macro> -->
 <!-- ========================================================================-->
 <!-- ===================== Material ============================================

File: description/robot.urdf.xacro (robot description, xacro)
@@ -2,11 +2,11 @@
 <robot xmlns:xacro="http://www.ros.org/wiki/xacro"  name="robot">
     <xacro:include filename="robot_core.xacro" />
-    <!-- <xacro:if value="$(arg use_ros2_control)">
+    <xacro:if value="$(arg use_ros2_control)">
         <xacro:include filename="ros2_control.xacro" />
     </xacro:if>
     <xacro:unless value="$(arg use_ros2_control)">
         <xacro:include filename="gazebo_control.xacro" />
-    </xacro:unless> -->
-    <xacro:include filename="gazebo_control.xacro" />
+    </xacro:unless>
+    <!-- <xacro:include filename="gazebo_control.xacro" /> -->
     <!-- <xacro:include filename="lidar.xacro"/> -->
     <xacro:include filename="camera.xacro"/>

File: description/robot_core.xacro (robot description, xacro)
@@ -6,4 +6,5 @@
     <xacro:include filename="$(find ${package_name})/description/common_sensors.urdf.xacro" />
     <xacro:include filename="$(find ${package_name})/description/andino_caster_macro.urdf.xacro" />
+    <xacro:include filename="inertial_macros.xacro" />
     <xacro:arg name="use_ros2_control" default="true" />
     <xacro:arg name="sim_mode" default="false" />
@@ -19,5 +20,4 @@
     <xacro:property name="sensor_yaml" value="$(arg yaml_config_dir)/sensors.yaml" />
     <xacro:property name="sensor_prop" value="${xacro.load_yaml(sensor_yaml)}" />
-    <xacro:include filename="inertial_macros.xacro" />
     <!-- Footprint -->
     <xacro:footprint wheel_props="${wheel_props}" />
@@ -54,5 +54,5 @@
     </gazebo>
     <!-- Wheels -->
-    <xacro:wheel prefix="right" reflect="-1"
+    <!-- <xacro:wheel prefix="right" reflect="-1"
         wheel_props="${wheel_props}"
         base_props="${base_props}">
@@ -61,16 +61,18 @@
         wheel_props="${wheel_props}"
         base_props="${base_props}">
-    </xacro:wheel>
+    </xacro:wheel> -->
     <!-- left wheel link -->
-    <!-- <joint name="left_wheel_joint" type="continuous">
+    <joint name="left_wheel_joint" type="continuous">
         <parent link="base_link" />
         <child link="left_wheel" />
-        <origin xyz="0 0.1 0.0" rpy="-${pi/2} 0 0" />
-        <axis xyz="0 0 1" />
+        <origin xyz="0 0.1 0.0" rpy="${pi/2} 0 0" />
+        <axis xyz="0 0 -1" />
     </joint>
     <link name="left_wheel">
         <visual>
             <geometry>
-                <cylinder radius="0.031" length="0.025" />
+                <!-- <cylinder radius="0.031" length="0.025" /> -->
+                <mesh
+                filename="file://$(find diff_robot)/meshes//components/wheel.stl" />
             </geometry>
             <material name="blue" />
@@ -87,16 +89,18 @@
     <gazebo reference="left_wheel">
         <material>Gazebo/Blue</material>
-    </gazebo> -->
+    </gazebo>
     <!-- right wheel link -->
-    <!-- <joint name="right_wheel_joint" type="continuous">
+    <joint name="right_wheel_joint" type="continuous">
         <parent link="base_link" />
         <child link="right_wheel" />
-        <origin xyz="0 -0.1 0.0" rpy="${pi/2} 0 0" />
-        <axis xyz="0 0 -1" />
+        <origin xyz="0 -0.1 0.0" rpy="-${pi/2} 0 0" />
+        <axis xyz="0 0 1" />
     </joint>
     <link name="right_wheel">
         <visual>
             <geometry>
-                <cylinder radius="0.031" length="0.025" />
+                <!-- <cylinder radius="0.031" length="0.025" /> -->
+                <mesh
+                filename="file://$(find diff_robot)/meshes//components/wheel.stl" />
             </geometry>
             <material name="blue" />
@@ -113,10 +117,10 @@
     <gazebo reference="right_wheel">
         <material>Gazebo/Blue</material>
-    </gazebo> -->
+    </gazebo>
     <!-- caster wheel link -->
-    <!-- <joint name="caster_wheel_joint" type="fixed">
+    <joint name="caster_wheel_joint" type="fixed">
         <parent link="chassis" />
         <child link="caster_wheel" />
-        <origin xyz="-0.03 0.0 -0.003" />
+        <origin xyz="-0.03 0.0 -0.0" />
     </joint>
     <link name="caster_wheel">
@@ -140,8 +144,8 @@
         <mu1 value="0.001" />
         <mu2 value="0.001" />
-    </gazebo> -->
-    <xacro:caster_wheel reflect="-1" use_fixed="$(arg use_fixed_caster)"
+    </gazebo>
+    <!-- <xacro:caster_wheel reflect="-1" use_fixed="$(arg use_fixed_caster)"
         wheel_props="${caster_wheel_props}">
-    </xacro:caster_wheel>
+    </xacro:caster_wheel> -->
     <xacro:laser prefix="rplidar" parent_link="chassis" sensor_prop="${sensor_prop}">
     </xacro:laser>

Commit message: for robot

File: description/andino_caster_macro.urdf.xacro (robot description, xacro)
@@ -29,10 +29,10 @@
             <xacro:if value="${scale != '' }">
               <mesh
-                filename="file://$(find diff_robot)/meshes/${robot_name}/${wheel_props['base']['mesh']}"
+                filename="package://diff_robot/meshes/${robot_name}/${wheel_props['base']['mesh']}"
                 scale="${scale}" />
             </xacro:if>
             <xacro:if value="${scale == '' }">
               <mesh
-                filename="file://$(find diff_robot)/meshes/${robot_name}/${wheel_props['base']['mesh']}" />
+                filename="package://diff_robot/meshes/${robot_name}/${wheel_props['base']['mesh']}" />
             </xacro:if>
           </geometry>
@@ -81,10 +81,10 @@
             <xacro:if value="${scale != '' }">
               <mesh
-                filename="file://$(find diff_robot)/meshes/${robot_name}/${wheel_props['hub']['mesh']}"
+                filename="package://diff_robot/meshes/${robot_name}/${wheel_props['hub']['mesh']}"
                 scale="${scale}" />
             </xacro:if>
             <xacro:if value="${scale == '' }">
               <mesh
-                filename="file://$(find diff_robot)/meshes/${robot_name}/${wheel_props['hub']['mesh']}" />
+                filename="package://diff_robot/meshes/${robot_name}/${wheel_props['hub']['mesh']}" />
             </xacro:if>
           </geometry>
@@ -144,10 +144,10 @@
             <xacro:if value="${scale != '' }">
               <mesh
-                filename="file://$(find diff_robot)/meshes/${robot_name}/${wheel_props['wheel']['mesh']}"
+                filename="package://diff_robot/meshes/${robot_name}/${wheel_props['wheel']['mesh']}"
                 scale="${scale}" />
             </xacro:if>
             <xacro:if value="${scale == '' }">
               <mesh
-                filename="file://$(find diff_robot)/meshes/${robot_name}/${wheel_props['wheel']['mesh']}" />
+                filename="package://diff_robot/meshes/${robot_name}/${wheel_props['wheel']['mesh']}" />
             </xacro:if>
           </geometry>

File: description/camera.xacro (robot description, xacro)
@@ -11,5 +11,5 @@
                 <box size="0.01 0.03 0.03"/>
             </geometry>
-            <material name="red"/>
+            <material name="black"/>
         </visual>
     </link>

File: description/common_macros.urdf.xacro (robot description, xacro)
@@ -271,5 +271,8 @@
   <material name="orange">
     <color rgba="1 0.3 0.1 1"/>
-</material>
+  </material>
+  <material name="white_1">
+    <color rgba="0.98 1 0.88 1"/>
+  </material>
 <!-- ========================================================================-->
 </robot>

File: description/common_sensors.urdf.xacro (robot description, xacro)
@@ -9,5 +9,5 @@
                     <origin xyz="0 0 0" rpy="0 0 ${pi}" />
                     <geometry>
-                        <mesh filename="file://$(find diff_robot)/meshes/sensors/${mesh}" />
+                        <mesh filename="package://diff_robot/meshes/sensors/${mesh}" />
                     </geometry>
                     <material name="dark_grey" />
@@ -54,5 +54,5 @@
                     <origin xyz="0 0 0" rpy="0 0 0" />
                     <geometry>
-                        <mesh filename="file://$(find diff_robot)/meshes/sensors/${mesh}" />
+                        <mesh filename="package://diff_robot/meshes/sensors/${mesh}" />
                     </geometry>
                     <material name="blue" />

File: description/robot_core.xacro (robot description, xacro)
@@ -7,6 +7,4 @@
     <xacro:include filename="$(find ${package_name})/description/andino_caster_macro.urdf.xacro" />
     <xacro:include filename="inertial_macros.xacro" />
-    <xacro:arg name="use_ros2_control" default="true" />
-    <xacro:arg name="sim_mode" default="false" />
     <xacro:arg name="yaml_config_dir" default="$(find ${package_name})/config/${robot_name}" />
     <xacro:property name="caster_wheel_yaml" value="$(arg yaml_config_dir)/caster_wheel.yaml" />
@@ -37,5 +35,5 @@
                 <box size="0.23 0.15 0.075" />
             </geometry>
-            <material name="white" />
+            <material name="white_1" />
         </visual>
         <collision>
@@ -46,5 +44,5 @@
             <material name="white" />
         </collision>
-        <xacro:inertial_box mass="0.5" x="0.3" y="0.3" z="0.15">
+        <xacro:inertial_box mass="1" x="0.3" y="0.3" z="0.15">
             <origin xyz="0.05 0 0.075" rpy="0 0 0" />
         </xacro:inertial_box>
@@ -66,5 +64,5 @@
         <parent link="base_link" />
         <child link="left_wheel" />
-        <origin xyz="0 0.1 0.0" rpy="${pi/2} 0 0" />
+        <origin xyz="0 0.095 0.0" rpy="${pi/2} 0 0" />
         <axis xyz="0 0 -1" />
     </joint>
@@ -73,8 +71,7 @@
             <geometry>
                 <!-- <cylinder radius="0.031" length="0.025" /> -->
-                <mesh
-                filename="file://$(find diff_robot)/meshes//components/wheel.stl" />
+                <mesh filename="package://diff_robot/meshes//components/wheel.stl" />
             </geometry>
-            <material name="blue" />
+            <material name="dark_grey" />
         </visual>
         <collision>
@@ -88,5 +85,5 @@
     </link>
     <gazebo reference="left_wheel">
-        <material>Gazebo/Blue</material>
+        <material>Gazebo/Black</material>
     </gazebo>
     <!-- right wheel link -->
@@ -94,5 +91,5 @@
         <parent link="base_link" />
         <child link="right_wheel" />
-        <origin xyz="0 -0.1 0.0" rpy="-${pi/2} 0 0" />
+        <origin xyz="0 -0.095 0.0" rpy="-${pi/2} 0 0" />
         <axis xyz="0 0 1" />
     </joint>
@@ -101,8 +98,9 @@
             <geometry>
                 <!-- <cylinder radius="0.031" length="0.025" /> -->
-                <mesh
-                filename="file://$(find diff_robot)/meshes//components/wheel.stl" />
+                <!-- <mesh
+                filename="file://$(find diff_robot)/meshes//components/wheel.stl" /> -->
+                <mesh filename="package://diff_robot/meshes//components/wheel.stl" />
             </geometry>
-            <material name="blue" />
+            <material name="dark_grey" />
         </visual>
         <collision>
@@ -116,5 +114,5 @@
     </link>
     <gazebo reference="right_wheel">
-        <material>Gazebo/Blue</material>
+        <material>Gazebo/Black</material>
     </gazebo>
     <!-- caster wheel link -->
@@ -122,12 +120,12 @@
         <parent link="chassis" />
         <child link="caster_wheel" />
-        <origin xyz="-0.03 0.0 -0.0" />
+        <origin xyz="-0.03 0.0 -0.008" />
     </joint>
     <link name="caster_wheel">
         <visual>
             <geometry>
-                <sphere radius="0.035" />
+                <sphere radius="0.025" />
             </geometry>
-            <material name="black" />
+            <material name="white" />
         </visual>
         <collision>

File: description/ros2_control.xacro (robot description, xacro)
@@ -1,15 +1,16 @@
 <?xml version="1.0"?>
 <robot xmlns:xacro="http://www.ros.org/wiki/xacro">
-     <xacro:unless value="$(arg sim_mode)">
+    <xacro:unless value="$(arg sim_mode)">
         <ros2_control name="RealRobot" type="system">
             <hardware>
-                <plugin>diffdrive_arduino/DiffDriveArduino</plugin>
+                <plugin>diffdrive_arduino/DiffDriveArduinoHardware</plugin>
                 <param name="left_wheel_name">left_wheel_joint</param>
                 <param name="right_wheel_name">right_wheel_joint</param>
                 <param name="loop_rate">30</param>
-                <param name="device">/dev/ttyUSB0</param>
+                <param name="device">/dev/ttyUSB_ARDUINO</param>
                 <param name="baud_rate">57600</param>
-                <param name="timeout">1000</param>
-                <param name="enc_counts_per_rev">525</param>
+                <param name="timeout_ms">1000</param>
+                <param name="enc_counts_per_rev_l">2273</param>
+                <param name="enc_counts_per_rev_r">2097</param>
             </hardware>
             <joint name="left_wheel_joint">
@@ -18,6 +19,6 @@
                     <param name="max">5</param>
                 </command_interface>
+                <state_interface name="position"/>
                 <state_interface name="velocity"/>
-                <state_interface name="position"/>
             </joint>
             <joint name="right_wheel_joint">
@@ -26,6 +27,6 @@
                     <param name="max">5</param>
                 </command_interface>
+                <state_interface name="position"/>
                 <state_interface name="velocity"/>
-                <state_interface name="position"/>
             </joint>
         </ros2_control>
@@ -41,6 +42,6 @@
                     <param name="max">5</param>
                 </command_interface>
+                <state_interface name="position"/>
                 <state_interface name="velocity"/>
-                <state_interface name="position"/>
             </joint>
             <joint name="right_wheel_joint">
@@ -49,6 +50,6 @@
                     <param name="max">5</param>
                 </command_interface>
+                <state_interface name="position"/>
                 <state_interface name="velocity"/>
-                <state_interface name="position"/>
             </joint>
         </ros2_control>
@@ -60,9 +61,3 @@
         </plugin>
     </gazebo>
-<!--
-    <gazebo>
-        <plugin name="gazebo_ros2_control" filename="libgazebo_ros2_control.so">
-            <parameters>$(find diff_robot)/config/my_controllers.yaml</parameters>
-        </plugin>
-    </gazebo> -->
 </robot>
