Commit message: clear code

File: description/andino_caster_macro.urdf.xacro (robot description, xacro)
@@ -62,5 +62,5 @@
         xyz="${wheel_props['base']['dx']} ${-wheel_props['base']['dy'] * locationright} ${wheel_props['base']['dz']}"
         rpy="0 0 0" />
-      <parent link="chassis" />
+      <parent link="caster_wheel_sp" />
       <child link="caster_base_link" />
       <axis xyz="0 0 1" />
@@ -115,5 +115,5 @@
           xyz="${wheel_props['hub']['dx']} ${-wheel_props['hub']['dy'] * locationright} ${wheel_props['hub']['dz']}"
           rpy="0 0 0" />
-        <parent link="chassis" />
+        <parent link="caster_wheel_sp" />
         <child link="caster_rotation_link" />
         <axis xyz="0 0 1" />
@@ -126,5 +126,5 @@
           xyz="${wheel_props['hub']['dx']} ${-wheel_props['hub']['dy'] * locationright} ${wheel_props['hub']['dz']}"
           rpy="0 0 0" />
-        <parent link="chassis" />
+        <parent link="caster_wheel_sp" />
         <child link="caster_rotation_link" />
         <axis xyz="0 0 1" />

File: description/camera.xacro (robot description, xacro)
@@ -4,13 +4,16 @@
         <parent link="chassis"/>
         <child link="camera_link"/>
-        <origin xyz="0.17 0 0.085" rpy = "0 0 0"/>
+        <origin xyz="-0.013 0 0.085" rpy = "0 0 0"/>
     </joint>
     <link name="camera_link">
         <visual>
             <geometry>
-                <box size="0.01 0.03 0.03"/>
+                <box size="0.015 0.07 0.02"/>
             </geometry>
-            <material name="red"/>
+            <material name="dark_grey"/>
         </visual>
+        <xacro:inertial_box mass="0.05" x="0.013" y="0.0" z="0.085">
+            <origin xyz="0.0 0 0.0" rpy="0 0 0" />
+        </xacro:inertial_box>
     </link>
     <joint name="camera_optical_joint" type="fixed">

File: description/common_macros.urdf.xacro (robot description, xacro)
@@ -13,5 +13,5 @@
                params="prefix reflect wheel_props base_props ">
   <xacro:property name="pos_x_joint"
-     value="${(base_props['base']['x_size']/2) - wheel_props['x_offset']}"/>
+     value="${wheel_props['x_offset']}"/>
   <xacro:property name="pos_y_joint"
     value="${(base_props['base']['y_size']/2) + wheel_props['y_offset'] + (wheel_props['length']/2)}"/>
@@ -158,5 +158,5 @@
           <box size="${base_prop['base']['x_size']} ${base_prop['base']['y_size']} ${base_prop['base']['z_size']}"/>
         </geometry>
-        <material name="blue" />
+        <material name="silver" />
       </visual>
     </xacro:if>
@@ -220,26 +220,4 @@
     </inertial>
   </xacro:macro>
-<!-- ===================== Sphere intertia xacro ===============================
-  params:
-  - m [float]: link mass;
-  - r [float]: sphere radius;
--->
-  <!-- <xacro:macro name="sphere_inertia" params="m r">
-    <inertial>
-      <mass value="${m}"/>
-      <inertia ixx="${2.0*m*(r*r)/5.0}" ixy="0.0" ixz="0.0" iyy="${2.0*m*(r*r)/5.0}" iyz="0.0" izz="${2.0*m*(r*r)/5.0}"/>
-    </inertial>
-  </xacro:macro> -->
-<!-- ===================== Default intertial xacro =============================
-  params:
-  - m [float]: link mass;
--->
-  <!-- <xacro:macro name="default_inertial" params="mass">
-    <inertial>
-      <mass value="${mass}"/>
-      <inertia ixx="1.0" ixy="0.0" ixz="0.0" iyy="1.0" iyz="0.0" izz="1.0"/>
-    </inertial>
-  </xacro:macro> -->
-<!-- ========================================================================-->
 <!-- ===================== Material ============================================
   RVIZ material RGBA definition.

File: description/common_sensors.urdf.xacro (robot description, xacro)
@@ -64,7 +64,7 @@
                     <geometry>
                         <box
-                            size="${sensor_prop['camera']['box_size']} ${sensor_prop['camera']['box_size']} ${sensor_prop['camera']['box_size']}" />
+                            size="${sensor_prop['camera']['x_size']} ${sensor_prop['camera']['y_size']} ${sensor_prop['camera']['z_size']}" />
                     </geometry>
-                    <material name="blue" />
+                    <material name="dark_grey" />
                 </visual>
             </xacro:if>
@@ -73,11 +73,11 @@
                 <geometry>
                     <box
-                        size="${sensor_prop['camera']['box_size']} ${sensor_prop['camera']['box_size']} ${sensor_prop['camera']['box_size']}" />
+                        size="${sensor_prop['camera']['x_size']} ${sensor_prop['camera']['y_size']} ${sensor_prop['camera']['z_size']}" />
                 </geometry>
             </collision>
             <xacro:box_inertia m="${sensor_prop['camera']['mass']}"
-                x="${sensor_prop['camera']['box_size']}"
-                y="${sensor_prop['camera']['box_size']}"
-                z="${sensor_prop['camera']['box_size']}"
+                x="${sensor_prop['camera']['x_size']}"
+                y="${sensor_prop['camera']['y_size']}"
+                z="${sensor_prop['camera']['z_size']}"
                 o_xyz="0 0 0"
                 o_rpy="0 0 0" />

File: description/robot.urdf.xacro (robot description, xacro)
@@ -10,7 +10,5 @@
         <xacro:include filename="gazebo_control.xacro" />
     </xacro:unless>
-    <!-- <xacro:include filename="gazebo_control.xacro" /> -->
-    <!-- <xacro:include filename="ros2_control.xacro" /> -->
     <!-- <xacro:include filename="lidar.xacro"/> -->
-    <xacro:include filename="camera.xacro"/>
+    <!-- <xacro:include filename="camera.xacro"/> -->
 </robot>

File: description/robot_core.xacro (robot description, xacro)
@@ -10,5 +10,5 @@
     <xacro:property name="caster_wheel_yaml" value="$(arg yaml_config_dir)/caster_wheel.yaml" />
     <xacro:property name="caster_wheel_props" value="${xacro.load_yaml(caster_wheel_yaml)}" />
-    <xacro:arg name="use_fixed_caster" default="True" />
+    <xacro:arg name="use_fixed_caster" default="False" />
     <xacro:arg name="use_real_ros_control" default="True" />
     <xacro:property name="base_yaml" value="$(arg yaml_config_dir)/base.yaml" />
@@ -27,9 +27,9 @@
         <parent link="base_link" />
         <child link="chassis" />
-        <origin xyz="-0.1 0.0 0.0" />
+        <origin xyz="0.05 0.0 0.04" />
     </joint>
     <link name="chassis">
         <visual>
-            <origin xyz="0.05 0.0 0.075" />
+            <origin xyz="-0.115 0.0 0.0375" />
             <geometry>
                 <box size="0.23 0.15 0.075" />
@@ -38,5 +38,5 @@
         </visual>
         <collision>
-            <origin xyz="0.05 0.0 0.075" />
+            <origin xyz="-0.115 0.0 0.0375" />
             <geometry>
                 <box size="0.23 0.15 0.075" />
@@ -44,7 +44,7 @@
             <material name="white" />
         </collision>
-        <xacro:inertial_box mass="0.5" x="0.3" y="0.3" z="0.15">
-            <origin xyz="0.05 0 0.075" rpy="0 0 0" />
-        </xacro:inertial_box>
+        <xacro:box_inertia m="0.1" x="0.23" y="0.15" z="0.075" o_xyz='-0.115 0.0 0.0375' o_rpy='0.0 0.0 0.0'>
+            <!-- <origin xyz="-0.115 0.0 0.0375" rpy="0 0 0" /> -->
+        </xacro:box_inertia>
     </link>
     <gazebo reference="chassis">
@@ -52,5 +52,5 @@
     </gazebo>
     <!-- Wheels -->
-    <!-- <xacro:wheel prefix="right" reflect="-1"
+    <xacro:wheel prefix="right" reflect="-1"
         wheel_props="${wheel_props}"
         base_props="${base_props}">
@@ -59,7 +59,7 @@
         wheel_props="${wheel_props}"
         base_props="${base_props}">
-    </xacro:wheel> -->
+    </xacro:wheel>
     <!-- left wheel link -->
-    <joint name="left_wheel_joint" type="continuous">
+    <!-- <joint name="left_wheel_joint" type="continuous">
         <parent link="base_link" />
         <child link="left_wheel" />
@@ -70,16 +70,16 @@
         <visual>
             <geometry>
-                <!-- <cylinder radius="0.031" length="0.025" /> -->
+                <cylinder radius="0.031" length="0.025" />
                 <mesh
                 filename="file://$(find diff_robot)/meshes//components/wheel.stl" />
             </geometry>
-            <material name="blue" />
+            <material name="dark_grey" />
         </visual>
         <collision>
             <geometry>
-                <sphere radius="0.031" />
+                <sphere radius="0.032" />
             </geometry>
         </collision>
-        <xacro:inertial_cylinder mass="0.1" length="0.025" radius="0.031">
+        <xacro:inertial_cylinder mass="0.03" length="0.025" radius="0.032">
             <origin xyz="0 0 0" rpy="0 0 0" />
         </xacro:inertial_cylinder>
@@ -87,7 +87,7 @@
     <gazebo reference="left_wheel">
         <material>Gazebo/Blue</material>
-    </gazebo>
+    </gazebo> -->
     <!-- right wheel link -->
-    <joint name="right_wheel_joint" type="continuous">
+    <!-- <joint name="right_wheel_joint" type="continuous">
         <parent link="base_link" />
         <child link="right_wheel" />
@@ -98,16 +98,15 @@
         <visual>
             <geometry>
-                <!-- <cylinder radius="0.031" length="0.025" /> -->
                 <mesh
                 filename="file://$(find diff_robot)/meshes//components/wheel.stl" />
             </geometry>
-            <material name="blue" />
+            <material name="dark_grey" />
         </visual>
         <collision>
             <geometry>
-                <sphere radius="0.031" />
+                <sphere radius="0.032" />
             </geometry>
         </collision>
-        <xacro:inertial_cylinder mass="0.1" length="0.025" radius="0.031">
+        <xacro:inertial_cylinder mass="0.03" length="0.025" radius="0.032">
             <origin xyz="0 0 0" rpy="0 0 0" />
         </xacro:inertial_cylinder>
@@ -115,15 +114,38 @@
     <gazebo reference="right_wheel">
         <material>Gazebo/Blue</material>
-    </gazebo>
+    </gazebo> -->
+    <!--support caster wheel link -->
+    <joint name="sp_caster_wheel_joint" type="fixed">
+        <parent link="chassis" />
+        <child link="caster_wheel_sp" />
+        <origin xyz="-0.18 0.0 0.0" />
+    </joint>
+    <link name="caster_wheel_sp">
+        <visual>
+            <origin xyz="0.0 0.0 -0.015" />
+            <geometry>
+                <box size="0.01 0.01 0.03" />
+            </geometry>
+            <material name="red" />
+        </visual>
+        <collision>
+            <geometry>
+                <box size="0.02 0.02 0.03" />
+            </geometry>
+        </collision>
+        <xacro:inertial_box mass="0.01" x="0.01" y="0.01" z="0.03">
+            <origin xyz="0 0 0" rpy="0 0 0" />
+        </xacro:inertial_box>
+    </link>
     <!-- caster wheel link -->
-    <joint name="caster_wheel_joint" type="fixed">
-        <parent link="chassis" />
+    <!-- <joint name="caster_wheel_joint" type="fixed">
+        <parent link="caster_wheel_sp" />
         <child link="caster_wheel" />
-        <origin xyz="-0.03 0.0 -0.0" />
+        <origin xyz="-0.0 0.0 -0.05" />
     </joint>
     <link name="caster_wheel">
         <visual>
             <geometry>
-                <sphere radius="0.035" />
+                <sphere radius="0.025" />
             </geometry>
             <material name="black" />
@@ -134,5 +156,5 @@
             </geometry>
         </collision>
-        <xacro:inertial_sphere mass="0.1" radius="0.025">
+        <xacro:inertial_sphere mass="0.01" radius="0.025">
             <origin xyz="0 0 0" rpy="0 0 0" />
         </xacro:inertial_sphere>
@@ -142,9 +164,11 @@
         <mu1 value="0.001" />
         <mu2 value="0.001" />
-    </gazebo>
-    <!-- <xacro:caster_wheel reflect="-1" use_fixed="$(arg use_fixed_caster)"
+    </gazebo> -->
+    <xacro:caster_wheel reflect="-1" use_fixed="$(arg use_fixed_caster)"
         wheel_props="${caster_wheel_props}">
-    </xacro:caster_wheel> -->
+    </xacro:caster_wheel>
     <xacro:laser prefix="rplidar" parent_link="chassis" sensor_prop="${sensor_prop}">
     </xacro:laser>
+    <xacro:camera_sensor parent_link="chassis" sensor_prop="${sensor_prop}">
+    </xacro:camera_sensor>
 </robot>

File: description/ros2_control.xacro (robot description, xacro)
@@ -42,6 +42,6 @@
                     <param name="max">5</param>
                 </command_interface>
+                <state_interface name="velocity"/>
                 <state_interface name="position"/>
-                <state_interface name="velocity"/>
             </joint>
             <joint name="right_wheel_joint">
@@ -50,6 +50,6 @@
                     <param name="max">5</param>
                 </command_interface>
+                <state_interface name="velocity"/>
                 <state_interface name="position"/>
-                <state_interface name="velocity"/>
             </joint>
         </ros2_control>

Commit message: update

File: description/andino_caster_macro.urdf.xacro (robot description, xacro)
@@ -173,4 +173,9 @@
       </collision>
     </link>
+    <gazebo reference="caster_wheel_link">
+      <material>Gazebo/White</material>
+      <mu1 value="0.001" />
+      <mu2 value="0.001" />
+    </gazebo>
     <xacro:if value="${use_fixed}">
       <joint name="caster_wheel_joint" type="fixed">

File: description/common_sensors.urdf.xacro (robot description, xacro)
@@ -45,4 +45,32 @@
             <axis xyz="0 1 0" />
         </joint>
+        <gazebo reference="${prefix}_laser_link">
+            <material>Gazebo/Black</material>
+            <sensor name="laser" type="ray">
+                <pose> 0 0 0 0 0 0 </pose>
+                <visualize>false</visualize>
+                <update_rate>10</update_rate>
+                <ray>
+                    <scan>
+                        <horizontal>
+                            <samples>360</samples>
+                            <min_angle>-3.14</min_angle>
+                            <max_angle>3.14</max_angle>
+                        </horizontal>
+                    </scan>
+                    <range>
+                        <min>0.3</min>
+                        <max>12</max>
+                    </range>
+                </ray>
+                <plugin name="laser_controller" filename="libgazebo_ros_ray_sensor.so">
+                    <ros>
+                        <remapping>~/out:=/scan</remapping>
+                    </ros>
+                    <output_type>sensor_msgs/LaserScan</output_type>
+                    <frame_name>rplidar_laser_link</frame_name>
+                </plugin>
+            </sensor>
+        </gazebo>
     </xacro:macro>
     <xacro:macro name="camera_sensor" params="parent_link sensor_prop">
@@ -88,7 +116,36 @@
             <origin
                 xyz="${sensor_prop['camera']['dx']} ${sensor_prop['camera']['dy']} ${sensor_prop['camera']['dz']}"
-                rpy="0 0 0" />
+                rpy="0 0.07 0" />
             <axis xyz="0 1 0" />
         </joint>
+        <joint name="camera_optical_joint" type="fixed">
+            <parent link="camera_link"/>
+            <child link="camera_link_optical"/>
+            <origin xyz="0.0 0 0.0" rpy = "${-pi/2} 0 ${-pi/2}"/>
+        </joint>
+        <link name="camera_link_optical"></link>
+        <gazebo reference="camera_link">
+            <material>Gazebo/Red</material>
+            <sensor name="camera" type="camera">
+                <pose> 0 0 0 0 0 0 </pose>
+                <visualize>true</visualize>
+                <update_rate>10</update_rate>
+                <camera>
+                    <horizontal_fov>1.089</horizontal_fov>
+                    <image>
+                        <format>R8G8B8</format>
+                        <width>640</width>
+                        <height>480</height>
+                    </image>
+                    <clip>
+                        <near>0.05</near>
+                        <far>8.0</far>
+                    </clip>
+                </camera>
+                <plugin name="camera_controller" filename="libgazebo_ros_camera.so">
+                    <frame_name>camera_link_optical</frame_name>
+                </plugin>
+            </sensor>
+        </gazebo>
     </xacro:macro>
 </robot>

File: description/robot_core.xacro (robot description, xacro)
@@ -10,5 +10,5 @@
     <xacro:property name="caster_wheel_yaml" value="$(arg yaml_config_dir)/caster_wheel.yaml" />
     <xacro:property name="caster_wheel_props" value="${xacro.load_yaml(caster_wheel_yaml)}" />
-    <xacro:arg name="use_fixed_caster" default="False" />
+    <xacro:arg name="use_fixed_caster" default="True" />
     <xacro:arg name="use_real_ros_control" default="True" />
     <xacro:property name="base_yaml" value="$(arg yaml_config_dir)/base.yaml" />
@@ -44,5 +44,5 @@
             <material name="white" />
         </collision>
-        <xacro:box_inertia m="0.1" x="0.23" y="0.15" z="0.075" o_xyz='-0.115 0.0 0.0375' o_rpy='0.0 0.0 0.0'>
+        <xacro:box_inertia m="1.0" x="0.23" y="0.15" z="0.075" o_xyz='-0.115 0.0 0.0375' o_rpy='0.0 0.0 0.0'>
             <!-- <origin xyz="-0.115 0.0 0.0375" rpy="0 0 0" /> -->
         </xacro:box_inertia>
